File: powertip-shiftreg.sch (KiCad schematic (older format))
At the start: 9 parts, among them P1 CONN_01X05, P2 CONN_01X03, U1 ICL7660, U2 74HC164, U3 HD44780

Commit message: - Board ist jetzt unter dem Display plaziert. - 3er Stecker hat jetzt VCC+, Contrast, VCC-
Connections:
- net GND: no longer P2.2 (P2)
- net Contrast: now reaches P1.3 (P3), U3.3 (Contrast)
- net Contrast: now also P2.2 (P2)
Changed lines of the file:
@@
-	1    0    0    -1
-$EndComp
-$Comp
-L GND #PWR03
-U 1 1 583879CC
-P 5450 4750
-F 0 "#PWR03" H 5450 4500 50  0001 C CNN
-F 1 "GND" H 5450 4600 50  0000 C CNN
-F 2 "" H 5450 4750 50  0000 C CNN
-F 3 "" H 5450 4750 50  0000 C CNN
-	1    5450 4750
 	1    0    0    -1
 $EndComp
@@
 Connection ~ 4950 4550
 Wire Wire Line
-	5650 4450 5450 4450
-Wire Wire Line
-	5450 4450 5450 4750
+	5650 4450 5200 4450
 $Comp
-L GND #PWR04
+L GND #PWR03
 U 1 1 58387F33
 P 3600 4750
-F 0 "#PWR04" H 3600 4500 50  0001 C CNN
+F 0 "#PWR03" H 3600 4500 50  0001 C CNN
 F 1 "GND" H 3600 4600 50  0000 C CNN
 F 2 "" H 3600 4750 50  0000 C CNN
@@
 Text Label 5000 4200 0    60   ~ 0
 VCC
+Text Label 5000 2400 0    60   ~ 0
+Contrast
+Text Label 5200 4450 0    60   ~ 0
+Contrast
 $EndSCHEMATC
